File: nRF51Socket.sch (EAGLE design)
At the start: 0 parts

Commit message: First revison.
Parts:
- added C2: 47nF, Nordic:CAP-403
- added C3: 1nF, Nordic:CAP-403
- added C4, C5, C6: 100nF, Nordic:CAP-403
- added C7, C8: 12pF, Nordic:CAP-403
- added FRAME1: FRAME-LETTERNO_PACKAGE, SparkFun-Aesthetics:FRAME-LETTERNO_PACKAGE
- added TC1: TC2030-IDC-NL, TagConnect:TC2030-IDC-NL
- added U1: QFN-48(52)BT-0.4-01-00, QFN-48(52)BT-0.4-01-00:QFN-48(52)BT-0.4-01-00
- added X1: 16MHz, Nordic:CRYSTAL-GND2520
Connections:
- new net 3.3V: C3.1, C4.1, C5.1, TC1.1, U1.AVDD, U1.AVDD$2, U1.VDD, U1.VDD$2
- new net GND: C2.2, C3.2, C4.2, C5.2, C6.2, C7.2, C8.2, TC1.5, U1.VSS, U1.VSS$2, U1.VSS$3, U1.VSS$4, X1.GND
- new net N$1: C2.1, U1.DEC2
- new net N$2: TC1.3
- new net N$6: C6.1, U1.DEC1
- new net N$7: C8.1, U1.XC1, X1.3
- new net N$8: C7.1, U1.XC2, X1.1
- new net SWDCLK: TC1.4, U1.SWDCLK
- new net SWDIO/!RESET: TC1.2, U1.SWDIO/!RESET

Commit message: Changed to 20pin jtag socket.
Parts:
- removed TC1: TC2030-IDC-NL, TagConnect:TC2030-IDC-NL
- added C18: 1uF, Nordic:CAP-403
- added FRAME2: FRAME-LETTERNO_PACKAGE, SparkFun-Aesthetics:FRAME-LETTERNO_PACKAGE
- added JP1: (no value), SparkFun-Connectors:M10X2
- added JP2: USB-MICROB, SparkFun-Connectors:USB-MICROB
- added U5: V_REG_LDOSMD, SparkFun-PowerIC:V_REG_LDOSMD
Connections:
- removed net N$2: TC1.3
- new net VBUS: JP1.19, JP2.VBUS, U5.EN, U5.IN
- net 3.3V: now also C18.1, JP1.1, U5.OUT; no longer TC1.1
- net GND: now also C18.2, JP1.10, JP1.12, JP1.14, JP1.16, JP1.18, JP1.20, JP1.4, JP1.6, JP1.8, JP2.GND, U5.GND; no longer TC1.5
- net SWDCLK: now also JP1.9; no longer TC1.4
- net SWDIO/!RESET: now also JP1.7; no longer TC1.2
